File: esp32_rf.brd (EAGLE design)
At the start: 160 x 100 mm, 31 parts, among them J1 TYPE-C-31-M-12, U1 ESP32-C3FH4, U2 AP2112K-3.3TRG1, U3 W25Q32FV, U4 USBLC6-2SC6, Y1 X1E000021017700, Y2 FC-135_32.7680KA-A0

Commit message: updates
Connections:
- new net N$13: C15.2, R5.1, U1.5, Y2.1
- net GND: now also C14.1, C15.1
- net N$12: now also R5.2
Changed lines of the file:
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@@
 <contactref element="S1" pad="4"/>
 <contactref element="S1" pad="3"/>
+<contactref element="C14" pad="1"/>
+<contactref element="C15" pad="1"/>
+<wire x1="-65.62" y1="-81.28" x2="-65.62" y2="-85.09" width="0" layer="19" extent="1-1"/>
+<wire x1="-56.3" y1="-69.85" x2="-65.62" y2="-81.28" width="0" layer="19" extent="1-1"/>
 <wire x1="-51.58" y1="-63.97" x2="-56.3" y2="-69.85" width="0" layer="19" extent="1-1"/>
 <wire x1="-47.48" y1="-63.97" x2="-51.58" y2="-63.97" width="0" layer="19" extent="1-1"/>
@@
 <contactref element="Y2" pad="2"/>
 <contactref element="C14" pad="2"/>
-<wire x1="-62.25" y1="-71.12" x2="-63.92" y2="-81.28" width="0" layer="19" extent="1-1"/>
+<contactref element="R5" pad="2"/>
+<wire x1="-63.92" y1="-77.47" x2="-63.92" y2="-81.28" width="0" layer="19" extent="1-1"/>
+<wire x1="-62.25" y1="-71.12" x2="-63.92" y2="-77.47" width="0" layer="19" extent="1-1"/>
 <wire x1="-25.31" y1="19.3" x2="-62.25" y2="-71.12" width="0" layer="19" extent="1-1"/>
 </signal>
+<signal name="N$13">
+<contactref element="U1" pad="5"/>
+<contactref element="Y2" pad="1"/>
+<contactref element="C15" pad="2"/>
+<contactref element="R5" pad="1"/>
+<wire x1="-65.62" y1="-77.47" x2="-63.92" y2="-85.09" width="0" layer="19" extent="1-1"/>
+<wire x1="-64.75" y1="-71.12" x2="-65.62" y2="-77.47" width="0" layer="19" extent="1-1"/>
+<wire x1="-25.31" y1="18.8" x2="-64.75" y2="-71.12" width="0" layer="19" extent="1-1"/>
+</signal>
 </signals>

Commit message: Updated schematic
Parts:
- added C16, C17, C18, C19, C20, C22, C23: 0.1uF, SparkFun-Capacitors:0603
- added D1: RED, SparkFun-LED:LED-0603
- added IC1: BMI055, BMI055:QFN50P300X450X100-16N
- added J2: 53261-0471, 53261-0471:MOLEX_53261-0471
- added L2: 2.2nH, SparkFun-Coils:0603
- added R10: 330, SparkFun-Resistors:0603
- added R11, R12: 4.7k, SparkFun-Resistors:0603
- added R6: 10k, SparkFun-Resistors:0603
- added R7: 22, SparkFun-Resistors:0603
- added R8, R9: 470, SparkFun-Resistors:0603
- added S2: MOMENTARY-SWITCH-SPST-SMD-4.6X2.8MM, SparkFun-Switches:TACTILE_SWITCH_SMD_4.6X2.8MM
- added U$1: MEANDER-ANT, Antennas:MEANDER-ANT
- added U5: BME280, BME280:PSON65P250X250X100-8N
- added U6: USBLC6-2SC6, USBLC6-2SC6:SOT95P280X145-6N
- moved U1 67.7 mm to (44.5, 11.4)
Connections:
- new net !CS: IC1.14, IC1.5, U1.16
- new net INT_ACCEL: IC1.16, U1.14
- new net INT_GYRO: C16.1, IC1.12, R6.1, S2.1, S2.2, U1.15
- new net LED_K: D1.C, R10.2
- new net MCU_LED: R10.1, U1.8
- new net MCU_RX: R8.1, U1.27
- new net MCU_TX: R9.1, U1.28
- new net MISO: IC1.10, IC1.15, U1.6
- new net MOSI: IC1.9, U1.13
- new net N$14: C22.1, J1.A4_B9, J1.B4_A9, L2.1
- new net N$15: R7.1, U1.12
- new net RX: J2.2, U6.4
- new net SCK: IC1.8, R7.2
- new net SCL: R11.1, U1.9, U5.4
- new net SDA: R12.1, U1.10, U5.3
- new net TX: J2.3, U6.6
- new net UART_RX: R8.2, U6.3
- new net UART_TX: R9.2, U6.1
- net 3.3V: now also C17.2, C18.2, C19.2, C20.2, D1.A, IC1.11, IC1.3, R11.2, R12.2, R6.2, U5.2, U5.6, U5.8
- net GND: now also C16.2, C17.1, C18.1, C19.1, C20.1, C22.2, C23.2, IC1.4, IC1.6, IC1.7, J2.4, J2.SH1, J2.SH2, S2.3, S2.4, U$1.GND, U5.1, U5.5, U5.7, U6.2; no longer J1.S1, J1.S2, J1.S3, J1.S4
- net V_USB: now also C23.1, J2.1, L2.2, U6.5; no longer J1.A4_B9, J1.B4_A9
Other:
- board size 160 x 100 mm -> 160 x 21.3 mm

Commit message: Design Files
Parts:
- removed RN1, RN2: 0R, SparkFun-Resistors:0805-ARV
- removed U3: W25Q32FV, SparkFun-IC-Memory:SOIC-8
- added D2: 1655, 1655:LED_1655
- added L3: WS2812B-2020, WS2812B-2020:WS2812B-2020
- moved C2 48.1 mm to (19.1, 36.8), turned to 225 degrees
- moved C1 44.6 mm to (20.3, 30.5), turned to 180 degrees
- moved U1 40.2 mm to (11.4, 34.3), turned to 315 degrees
- moved Y1 36.1 mm to (16.5, 39.4), turned to 225 degrees
- moved J1 35.7 mm to (12.7, 2.03)
- moved U$1 24.5 mm to (6.22, 43.8)
Connections:
- removed net N$10: RN1.5, U1.23
- removed net N$11: RN2.5, U1.24
- removed net N$7: RN1.8, U1.19
- removed net N$8: RN1.7, U1.20
- removed net N$9: RN1.6, U1.22
- removed net SPICLK: RN1.3, U3.6
- removed net SPICS0: U1.21, U3.1
- removed net SPID: RN1.4, U3.5
- removed net SPIHD: RN1.1, U3.7
- removed net SPIQ: RN2.4, U3.2
- removed net SPIWP: RN1.2, U3.3
- new net VDD: D2.3
- new net VSS: D2.1
- net 3.3V: no longer RN2.1, RN2.2, RN2.3, RN2.6, RN2.7, RN2.8
- net GND: no longer U3.4
- net VDD_SPI: no longer U3.8
Other:
- board size 160 x 21.3 mm -> 25.4 x 49 mm
