File: esp32_rf.sch (EAGLE design)
At the start: 31 parts, among them J1 TYPE-C-31-M-12, U1 ESP32-C3FH4, U2 AP2112K-3.3TRG1, U3 W25Q32FV, U4 USBLC6-2SC6, Y1 X1E000021017700, Y2 FC-135_32.7680KA-A0

Commit message: updates
Connections:
- new net N$13: C15.2, R5.1, U1.XTAL_32K_N, Y2.1
- net GND: now also C14.1, C15.1
- net N$12: now also R5.2
Other:
- note added: "USB"
- moved on the sheet: C14
Changed lines of the file:
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@@
 <part name="C14" library="SparkFun-Capacitors" library_urn="urn:adsk.eagle:library:510" deviceset="12PF" device="-0603-50V-5%" package3d_urn="urn:adsk.eagle:package:37414/1" value="8pF"/>
 <part name="C15" library="SparkFun-Capacitors" library_urn="urn:adsk.eagle:library:510" deviceset="12PF" device="-0603-50V-5%" package3d_urn="urn:adsk.eagle:package:37414/1" value="8pF"/>
+<part name="GND17" library="SparkFun-PowerSymbols" library_urn="urn:adsk.eagle:library:530" deviceset="GND" device=""/>
 </parts>
 <sheets>
@@
 <instance part="R4" gate="G$1" x="12.7" y="147.32" smashed="yes" rot="R90">
 <attribute name="NAME" x="11.684" y="151.384" size="1.016" layer="95" font="vector" ratio="20" rot="R180" align="bottom-center"/>
-<attribute name="VALUE" x="14.224" y="147.32" size="1.778" layer="96" font="vector" rot="R90" align="top-center"/>
+<attribute name="VALUE" x="11.176" y="143.256" size="1.016" layer="96" font="vector" ratio="20" rot="R180" align="top-center"/>
 </instance>
 <instance part="SUPPLY11" gate="G$1" x="12.7" y="160.02" smashed="yes">
@@
 </instance>
 <instance part="Y2" gate="G$1" x="27.94" y="83.82" smashed="yes" rot="R90">
-<attribute name="NAME" x="21.83455" y="78.73213125" size="1.27196875" layer="95" rot="R90"/>
-<attribute name="VALUE" x="35.58273125" y="78.724840625" size="1.273790625" layer="96" rot="R90"/>
+<attribute name="NAME" x="26.67786875" y="90.66855" size="1.016" layer="95" font="vector" ratio="20" rot="R180"/>
+<attribute name="VALUE" x="35.575159375" y="80.54073125" size="1.016" layer="96" font="vector" ratio="20" rot="R180"/>
 </instance>
 <instance part="R5" gate="G$1" x="40.64" y="83.82" smashed="yes" rot="R90">
-<attribute name="NAME" x="39.116" y="83.82" size="1.778" layer="95" font="vector" rot="R90" align="bottom-center"/>
-<attribute name="VALUE" x="42.164" y="83.82" size="1.778" layer="96" font="vector" rot="R90" align="top-center"/>
-</instance>
-<instance part="C14" gate="G$1" x="15.494" y="94.488" smashed="yes" rot="R90">
-<attribute name="NAME" x="13.208" y="96.139" size="1.016" layer="95" font="vector" ratio="20" rot="R180"/>
-<attribute name="VALUE" x="17.78" y="95.885" size="1.016" layer="96" font="vector" ratio="20" rot="R180"/>
+<attribute name="NAME" x="41.656" y="88.138" size="1.016" layer="95" font="vector" ratio="20" rot="R180" align="bottom-center"/>
+<attribute name="VALUE" x="42.164" y="79.756" size="1.016" layer="96" font="vector" ratio="20" rot="R180" align="top-center"/>
+</instance>
+<instance part="C14" gate="G$1" x="15.24" y="93.98" smashed="yes" rot="R90">
+<attribute name="NAME" x="12.954" y="95.631" size="1.016" layer="95" font="vector" ratio="20" rot="R180"/>
+<attribute name="VALUE" x="17.526" y="95.377" size="1.016" layer="96" font="vector" ratio="20" rot="R180"/>
 </instance>
 <instance part="C15" gate="G$1" x="15.748" y="73.66" smashed="yes" rot="R90">
 <attribute name="NAME" x="13.462" y="75.311" size="1.016" layer="95" font="vector" ratio="20" rot="R180"/>
 <attribute name="VALUE" x="18.034" y="75.057" size="1.016" layer="96" font="vector" ratio="20" rot="R180"/>
+</instance>
+<instance part="GND17" gate="1" x="5.08" y="62.992" smashed="yes">
+<attribute name="VALUE" x="4.826" y="62.484" size="1.016" layer="96" font="vector" ratio="20" align="top-center"/>
 </instance>
 </instances>
@@
 <wire x1="7.62" y1="109.22" x2="12.7" y2="109.22" width="0.1524" layer="91"/>
 <junction x="12.7" y="109.22"/>
+</segment>
+<segment>
+<pinref part="GND17" gate="1" pin="GND"/>
+<pinref part="C14" gate="G$1" pin="1"/>
+<wire x1="5.08" y1="65.532" x2="5.08" y2="73.66" width="0.1524" layer="91"/>
+<wire x1="5.08" y1="73.66" x2="5.08" y2="93.98" width="0.1524" layer="91"/>
+<wire x1="5.08" y1="93.98" x2="10.16" y2="93.98" width="0.1524" layer="91"/>
+<pinref part="C15" gate="G$1" pin="1"/>
+<wire x1="10.668" y1="73.66" x2="5.08" y2="73.66" width="0.1524" layer="91"/>
+<junction x="5.08" y="73.66"/>
 </segment>
 </net>
@@
 <wire x1="43.18" y1="111.76" x2="43.18" y2="93.98" width="0.1524" layer="91"/>
 <pinref part="Y2" gate="G$1" pin="2"/>
-<wire x1="43.18" y1="93.98" x2="27.94" y2="93.98" width="0.1524" layer="91"/>
+<wire x1="43.18" y1="93.98" x2="40.64" y2="93.98" width="0.1524" layer="91"/>
 <pinref part="C14" gate="G$1" pin="2"/>
-<wire x1="27.94" y1="93.98" x2="18.034" y2="93.98" width="0.1524" layer="91"/>
-<wire x1="18.034" y1="93.98" x2="18.034" y2="94.488" width="0.1524" layer="91"/>
+<wire x1="40.64" y1="93.98" x2="27.94" y2="93.98" width="0.1524" layer="91"/>
+<wire x1="27.94" y1="93.98" x2="17.78" y2="93.98" width="0.1524" layer="91"/>
 <junction x="27.94" y="93.98"/>
+<pinref part="R5" gate="G$1" pin="2"/>
+<wire x1="40.64" y1="88.9" x2="40.64" y2="93.98" width="0.1524" layer="91"/>
+<junction x="40.64" y="93.98"/>
+</segment>
+</net>
+<net name="N$13" class="0">
+<segment>
+<pinref part="U1" gate="G$1" pin="XTAL_32K_N"/>
+<wire x1="78.74" y1="109.22" x2="50.546" y2="109.22" width="0.1524" layer="91"/>
+<pinref part="Y2" gate="G$1" pin="1"/>
+<wire x1="50.546" y1="109.22" x2="50.546" y2="73.66" width="0.1524" layer="91"/>
+<wire x1="50.546" y1="73.66" x2="40.64" y2="73.66" width="0.1524" layer="91"/>
+<pinref part="C15" gate="G$1" pin="2"/>
+<wire x1="40.64" y1="73.66" x2="27.94" y2="73.66" width="0.1524" layer="91"/>
+<wire x1="27.94" y1="73.66" x2="18.288" y2="73.66" width="0.1524" layer="91"/>
+<junction x="27.94" y="73.66"/>
+<pinref part="R5" gate="G$1" pin="1"/>
+<wire x1="40.64" y1="78.74" x2="40.64" y2="73.66" width="0.1524" layer="91"/>
+<junction x="40.64" y="73.66"/>
 </segment>
 </net>
@@
 <plain>
 <text x="40.64" y="104.14" size="5.08" layer="94" font="vector" ratio="20">Power Supply</text>
+<text x="48.26" y="167.64" size="5.08" layer="94" font="vector" ratio="20">USB</text>
 </plain>
 <instances>

Commit message: Updated schematic
Parts:
- added C16, C17, C18, C19, C20, C22, C23: 0.1uF, SparkFun-Capacitors:0.1UF-0603-25V-(+80/-20%)
- added D1: RED, SparkFun-LED:LED0603
- added IC1: BMI055, BMI055:BMI055
- added J2: 53261-0471, 53261-0471:53261-0471
- added L2: 2.2nH, SparkFun-Coils:INDUCTOR-0603-33NH
- added R10: 330, SparkFun-Resistors:330OHM-0603-1/10W-1%
- added R11, R12: 4.7k, SparkFun-Resistors:4.7KOHM-0603-1/10W-1%
- added R6: 10k, SparkFun-Resistors:10KOHM-0603-1/10W-1%
- added R7: 22, SparkFun-Resistors:22OHM-0603-1/10W-1%
- added R8, R9: 470, SparkFun-Resistors:470OHM-0603-1/10W-1%
- added S2: MOMENTARY-SWITCH-SPST-SMD-4.6X2.8MM, SparkFun-Switches:MOMENTARY-SWITCH-SPST-SMD-4.6X2.8MM
- added U$1: MEANDER-ANT, Antennas:MEANDER-ANT
- added U5: BME280, BME280:BME280
- added U6: USBLC6-2SC6, USBLC6-2SC6:USBLC6-2SC6
Connections:
- new net !CS: IC1.CSB1, IC1.CSB2, U1.GPIO10
- new net INT_ACCEL: IC1.INT1, U1.GPIO8
- new net INT_GYRO: C16.1, IC1.INT3, R6.1, S2.1, U1.GPIO9
- new net LED_K: D1.C, R10.2
- new net MCU_LED: R10.1, U1.GPIO3
- new net MCU_RX: R8.1, U1.U0RXD
- new net MCU_TX: R9.1, U1.U0TXD
- new net MISO: IC1.SDO1, IC1.SDO2, U1.GPIO2
- new net MOSI: IC1.SDX, U1.MTDO
- new net N$14: C22.1, J1.VBUS, L2.1
- new net N$15: R7.1, U1.MTCK
- new net RX: J2.2, U6.I/O2_OUT
- new net SCK: IC1.SCX, R7.2
- new net SCL: R11.1, U1.MTMS, U5.SCK
- new net SDA: R12.1, U1.MTDI, U5.SDI
- new net TX: J2.3, U6.I/O1_OUT
- new net UART_RX: R8.2, U6.I/O2_IN
- new net UART_TX: R9.2, U6.I/O1_IN
- net 3.3V: now also C17.2, C18.2, C19.2, C20.2, D1.A, IC1.VDD, IC1.VDDIO, R11.2, R12.2, R6.2, U5.CSB, U5.VDD, U5.VDDIO
- net GND: now also C16.2, C17.1, C18.1, C19.1, C20.1, C22.2, C23.2, IC1.GNDA, IC1.GNDIO, IC1.PS, J2.4, J2.SHIELD, S2.2, U$1.GND, U5.GND, U5.SDO, U6.GND; no longer J1.SHIELD
- net V_USB: now also C23.1, J2.1, L2.2, U6.VBUS; no longer J1.VBUS

Commit message: Design Files
Parts:
- removed RN1, RN2: 0R, SparkFun-Resistors:1KOHM-ARRAY(4)-0805_ARV-1/10W-5%
- removed U3: W25Q32FV, SparkFun-IC-Memory:W25Q32FVSS
- added D2: 1655, 1655:1655
- added L3: WS2812B-2020, WS2812B-2020:WS2812B-2020
Connections:
- removed net N$10: RN1D.2, U1.SPID
- removed net N$11: RN2D.2, U1.SPIQ
- removed net N$7: RN1A.2, U1.SPIHD
- removed net N$8: RN1B.2, U1.SPIWP
- removed net N$9: RN1C.2, U1.SPICLK
- removed net SPICLK: RN1C.1, U3.SCK
- removed net SPICS0: U1.SPICS0, U3.!CS!
- removed net SPID: RN1D.1, U3.SI(D0)
- removed net SPIHD: RN1A.1, U3.!HOLD!(D3)
- removed net SPIQ: RN2D.1, U3.SO(D1)
- removed net SPIWP: RN1B.1, U3.!WP!(D2)
- net 3.3V: no longer RN2A.1, RN2A.2, RN2B.1, RN2B.2, RN2C.1, RN2C.2
- net GND: no longer U3.GND
- net VDD_SPI: no longer U3.VCC
